File: Hardware/LilyPad-E-Sewing-Kit.sch (EAGLE design)
At the start: 50 parts

Commit message: Fixed labeling on board.
Parts:
- added JP2: LOGO-SFESK, SparkFun-Aesthetics:LOGO-SFESK
Other:
- note added: "L. Buechley, N.Seidle, P. Lewis T. Klopfenstein"
- note added: "v13"
- note removed: "L. Buechley N.Seidle P. Lewis"
Changed lines of the file:
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@@
 <part name="JP1" library="SparkFun" deviceset="FIDUCIAL" device="1X2"/>
 <part name="U$8" library="SparkFun-Aesthetics" deviceset="OSHW-LOGO" device="S"/>
-<part name="FRAME1" library="SparkFun-Aesthetics" deviceset="FRAME-LETTER" device=""/>
 <part name="GND1" library="SparkFun-Aesthetics" deviceset="GND" device=""/>
 <part name="P+1" library="SparkFun-Aesthetics" deviceset="VCC" device=""/>
 <part name="P+2" library="SparkFun-Aesthetics" deviceset="VCC" device=""/>
 <part name="P+3" library="SparkFun-Aesthetics" deviceset="VCC" device=""/>
+<part name="FRAME1" library="SparkFun-Aesthetics" deviceset="FRAME-LETTER" device=""/>
+<part name="JP2" library="SparkFun-Aesthetics" deviceset="LOGO-SFE" device="SK"/>
 </parts>
 <sheets>
@@
 <wire x1="50.8" y1="0" x2="50.8" y2="22.86" width="0.2032" layer="94"/>
 <circle x="53.34" y="106.68" radius="27.4743" width="0.2032" layer="94"/>
-<text x="177.8" y="-35.56" size="1.778" layer="95">L. Buechley
-N.Seidle
-P. Lewis
-</text>
+<text x="182.88" y="-33.02" size="1.778" layer="95">L. Buechley, N.Seidle, P. Lewis
+T. Klopfenstein</text>
 <text x="167.64" y="137.16" size="1.778" layer="97">Changes to V13</text>
 <text x="172.72" y="132.08" size="1.778" layer="97">Rotated Lilypad silk
 Added OSHW and SFE flame</text>
+<text x="246.38" y="-33.02" size="1.778" layer="97">v13</text>
 </plain>
 <instances>
@@
 <instance part="U$7" gate="G$1" x="27.94" y="83.82"/>
 <instance part="JP1" gate="G$1" x="246.38" y="-7.62"/>
-<instance part="U$8" gate="G$1" x="134.62" y="-25.4"/>
-<instance part="FRAME1" gate="G$1" x="2.54" y="-40.64"/>
-<instance part="FRAME1" gate="G$2" x="149.86" y="-40.64"/>
+<instance part="U$8" gate="G$1" x="137.16" y="-30.48"/>
 <instance part="GND1" gate="1" x="25.4" y="71.12"/>
 <instance part="P+1" gate="1" x="99.06" y="127" rot="R270"/>
 <instance part="P+2" gate="1" x="231.14" y="96.52" rot="R270"/>
 <instance part="P+3" gate="1" x="233.68" y="71.12" rot="R270"/>
+<instance part="FRAME1" gate="G$1" x="7.62" y="-40.64"/>
+<instance part="FRAME1" gate="G$2" x="154.94" y="-40.64"/>
+<instance part="JP2" gate="G$1" x="248.92" y="-15.24"/>
 </instances>
 <busses>
